Commit message: WIP: This one works from the GUI, but not when I send commands from the command line.

File: urdf/my-simple-robot.urdf.xacro (robot description, xacro)
@@ -1,4 +1,4 @@
 <?xml version="1.0"?>
-<robot name="simple-robot" xmlns:xacro="http://ros.org/wiki/xacro">
+<robot name="simple_robot" xmlns:xacro="http://ros.org/wiki/xacro">
   <material name="white">
     <color rgba="1 1 1 0.9"/>
@@ -63,29 +63,20 @@
     <parent link="robot_base"/>
     <child link="robot_arm"/>
-    <origin rpy="0 0.66 0" xyz="0 0.1 0.45"/>
+    <origin rpy="0 0 0" xyz="0 0.1 0.45"/>
     <axis rpy="0 0 0" xyz="0 1 0"/>
-    <limit effort="10.0" lower="-3" upper="3" velocity="0.5"/>
-    <dynamics damping="0.001" friction="0.0001"/>
+    <limit effort="100.0" lower="-3" upper="3" velocity="100.0"/>
+    <dynamics damping="0.2" friction="0.001"/>
   </joint>
-  <ros2_control name="IgnitionSystem" type="system">
-    <hardware>
-      <plugin>ign_ros2_control/IgnitionSystem</plugin>
-    </hardware>
-    <joint name="the_joint">
-      <command_interface name="position">
-        <param name="min">-1</param>
-        <param name="max">1</param>
-      </command>
-      <state_interface name="position" />
-      <state_interface name="velocity"/>
-      <state_interface name="effort"/>
-    </joint>
-  </ros2_control>
   <gazebo>
-    <plugin filename="libign_ros2_control-system.so" name="ign_ros2_control::IgnitionROS2ControlPlugin">
-      <robot_param>robot_description</robot_param>
-      <robot_param_node>robot_state_publisher</robot_param_node>
-      <parameters>$(find ignition_ros2_control_test)/config/controller.yaml</parameters>
-    </plugin>
+    <plugin filename="ignition-gazebo-joint-position-controller-system" name="ignition::gazebo::systems::JointPositionController">
+      <joint_name>the_joint</joint_name>
+		  <p_gain>10000</p_gain>
+		  <i_gain>0.1</i_gain>
+		  <d_gain>5000</d_gain>
+		  <i_max>1</i_max>
+		  <i_min>-1</i_min>
+      <cmd_max>1000</cmd_max>
+      <cmd_min>-1000</cmd_min>
+		</plugin>
   </gazebo>
 </robot>
